File: MaimaiLed.kicad_sch (KiCad schematic)
At the start: 10 parts, among them J1 ConnLeft, J2 ConnRightNP

Commit message: Updated Readme and project schematic
Other:
- title: (none) -> Maimai LED - ILM-R1 compatible
- moved on the sheet: H1
Changed lines of the file:
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@@
 	(generator_version "8.0")
 	(paper "A4")
+	(title_block
+		(title "Maimai LED - ILM-R1 compatible")
+		(date "2024-10-05")
+		(rev "1.00")
+	)
 	(junction
 		(at 189.23 63.5)
@@
 	(symbol
 		(lib_id "Mechanical:MountingHole")
-		(at 121.92 36.83 0)
+		(at 114.3 36.83 0)
 		(unit 1)
 		(exclude_from_sim yes)
@@
 		(fields_autoplaced yes)
 		(property "Reference" "H1"
-			(at 124.46 35.5599 0)
+			(at 116.84 35.5599 0)
 			(effects
 				(font
@@
 		)
 		(property "Value" "MountingHole"
-			(at 124.46 38.0999 0)
+			(at 116.84 38.0999 0)
 			(effects
 				(font
@@
 		)
 		(property "Footprint" "MountingHole:MountingHole_3.2mm_M3"
-			(at 121.92 36.83 0)
+			(at 114.3 36.83 0)
 			(effects
 				(font
@@
 		)
 		(property "Datasheet" "~"
-			(at 121.92 36.83 0)
+			(at 114.3 36.83 0)
 			(effects
 				(font
@@
 		)
 		(property "Description" "Mounting Hole without connection"
-			(at 121.92 36.83 0)
-			(effects
-				(font
+			(at 114.3 36.83 0)
+			(effects
+				(font
